Commit message: lidarpositioning

File: src/vehicle_simulator/urdf/robot.urdf.xacro (robot description, xacro)
@@ -165,5 +165,5 @@
   // Lidar Joint
   <joint name="lidar_joint" type="fixed">
-    <origin xyz="0.15 0.0 0.1" rpy="0.0 0.0 0.0"/>
+    <origin xyz="0.0 0.0 0.05" rpy="0.0 0.0 0.0"/>
     <parent link="chassis"/>
     <child link="lidar"/>
